File: 2fer.kicad_pcb (KiCad board)
At the start: 2 copper layers, 50.8 x 22.9 mm, 6 parts, among them J1 feather long, J2 feather short

Commit message: Revision 1
Parts:
- added SW1: SW_Push, Button_Switch_Keyboard:SW_Cherry_MX_1.00u_PCB, F.Cu at (43.5, 31.8)
- added SW2: SW_Push, Button_Switch_Keyboard:SW_Cherry_MX_1.00u_PCB, F.Cu at (63.5, 31.8)
- added SW4: SW_SPDT, footprints:Switch-SPST_CSS-1210MC, B.Cu at (30.8, 35.2)
Routing:
- net /F5: track 0.00 -> 24.2 mm
- net /F4: track 0.00 -> 20.6 mm
- net /EN: track 0.00 -> 20.6 mm
- net /F3: track 0.00 -> 19.6 mm
- net GND: track 0.00 -> 15.3 mm
Other:
- board text added: "DFU"
- board text added: "TAHNOK"
- board text removed: "FREE"
